Commit message: t1 should start with lower noise_std

File: legged_gym/robots/g1/g1_15dof.urdf (robot description, URDF)
Before this commit: robot g1_15dof, 33 links, 32 joints
Joints:
- joint left_ankle_pitch_joint: origin xyz=0 -9.4445E-05 -0.30001 rpy=0 -1.57 0 -> xyz=0 -9.4445E-05 -0.30001 rpy=0 0 0
- joint right_ankle_pitch_joint: origin xyz=0 9.4445E-05 -0.30001 rpy=0 -1.57 0 -> xyz=0 9.4445E-05 -0.30001 rpy=0 0 0
