Commit message: you pretrain with plane, then start t1_odom_neg

File: legged_gym/robots/T1/T1_legs.urdf (robot description, URDF)
Before this commit: robot T1, 24 links, 23 joints
Joints:
- joint Head_pitch: origin xyz=0 0 0.06185 rpy=0 0 0 -> xyz=0 0 0.06185 rpy=0 0.785 0
- joint Left_Elbow_Yaw: origin xyz=0 0.1471 0 rpy=0 0 0 -> xyz=0 0.1471 0 rpy=0 0 -1
- joint Left_Shoulder_Pitch: origin xyz=0.0575 0.1063 0.219 rpy=0 0.00088113 0 -> xyz=0.0575 0.1063 0.219 rpy=0 0 0
- joint Left_Shoulder_Roll: origin xyz=0 0.047 0 rpy=0 0 0 -> xyz=0 0.047 0 rpy=-1.3 0 0
- joint Right_Elbow_Yaw: origin xyz=0 -0.1471 0 rpy=0 0 0 -> xyz=0 -0.1471 0 rpy=0 0 1
- joint Right_Shoulder_Pitch: origin xyz=0.0575 -0.1063 0.219 rpy=0 0.00088113 0 -> xyz=0.0575 -0.1063 0.219 rpy=0 0 0
- joint Right_Shoulder_Roll: origin xyz=0 -0.047 0 rpy=0 0 0 -> xyz=0 -0.047 0 rpy=1.3 0 0
